File: Board1.0/CruiseController.sch (KiCad schematic (older format))
At the start: 56 parts, among them J1 USB_B_Micro, J2 Conn_02x09_Top_Bottom, U3 TLV9064IRTER, U4 TS5A23157RSER, U5 MIC5225, U6 MCP2562-E-MF, U7 STM32L433CCUx, Y1 32.768

Commit message: Readability
Other:
- note added: "Power Budget (Target)\nSTM32: 10mA (1-2mA)\nTLV9064: 40mA ea + 2mAQc (6mA)\nMCP2562: 10mA (5mA)\nRGB: 30mA (Varies)\n"
- note removed: "Power Budget\nSTM32: 10mA\nTLV9064: 40mA ea + 2mAQc\nMCP2562: 10mA\nRGB: 30mA\n"
Changed lines of the file:
@@
 	1    0    0    -1
 $EndComp
-Text Notes 5525 5200 0    50   ~ 0
-Power Budget\nSTM32: 10mA\nTLV9064: 40mA ea + 2mAQc\nMCP2562: 10mA\nRGB: 30mA\n
+Text Notes 5000 5425 0    50   ~ 0
+Power Budget (Target)\nSTM32:    10mA (1-2mA)\nTLV9064:  40mA ea + 2mAQc (6mA)\nMCP2562: 10mA (5mA)\nRGB:      30mA (Varies)\n
 $Comp
 L Device:R_Small R8
