File: Board3.0/CruiseController.sch (KiCad schematic (older format))
At the start: 55 parts, among them J1 USB_B_Micro, J2 Conn_02x09_Top_Bottom, U1 ADG884, U3 TLV9064IRTER, U5 MIC5225, U6 MCP2562-E-MF, U7 STM32L433CCUx, Y1 32.768

Commit message: Update v3
Parts:
- R1: value 10k -> 2.2k
- U5: symbol MargoGeneral:MIC5225 -> CruiseController-rescue:MIC5225-MargoGeneral
Connections:
- net GND: no longer U3.4 (-)
- net at U3.5: now also U3.4 (-)
- no-connect marks 21 -> 20
Other:
- moved on the sheet: U3B
Changed lines of the file:
@@
 EESchema Schematic File Version 4
 LIBS:CruiseController-cache
-EELAYER 29 0
+EELAYER 30 0
 EELAYER END
 $Descr USLetter 11000 8500
@@
 	9300 1275 9725 1275
 $Comp
-L MargoGeneral:MIC5225 U5
+L CruiseController-rescue:MIC5225-MargoGeneral U5
 U 1 1 5DC6F376
 P 5375 4650
@@
 P 7875 1925
 F 0 "R1" V 7800 1950 50  0000 C CNN
-F 1 "10k" V 7875 1925 50  0000 C CNN
+F 1 "2.2k" V 7875 1925 50  0000 C CNN
 F 2 "Resistor_SMD:R_0603_1608Metric" H 7875 1925 50  0001 C CNN
 F 3 "~" H 7875 1925 50  0001 C CNN
@@
 Text Notes 5525 4750 0    50   ~ 0
 150mA
-Wire Wire Line
-	4625 4400 4850 4400
 Text GLabel 2025 3300 0    50   Input ~ 0
 TTAIN
@@
 $EndComp
 Connection ~ 5275 4400
-Connection ~ 4850 4400
-Text GLabel 4625 4400 0    50   Input ~ 0
+Text GLabel 4650 4400 0    50   Input ~ 0
 VIN
 $Comp
@@
 Connection ~ 3725 3575
 Connection ~ 3725 2725
-Connection ~ 3300 4600
-Wire Wire Line
-	3300 4400 3300 4600
-Wire Wire Line
-	3400 4400 3300 4400
-Wire Wire Line
-	3300 4600 3300 4650
-Wire Wire Line
-	3400 4600 3300 4600
+Wire Wire Line
+	3150 5400 3150 5550
+Wire Wire Line
+	3250 5400 3150 5400
 $Comp
 L CruiseController-rescue:TLV9064IRTER-VeridianDesigns-CruiseController-rescue U3
 U 2 1 5DCBC2C3
-P 3700 4500
-F 0 "U3" H 3700 4867 50  0000 C CNN
-F 1 "TLV9064IRTER" H 3700 4776 50  0000 C CNN
-F 2 "Package_DFN_QFN:QFN-16-1EP_3x3mm_P0.5mm_EP1.7x1.7mm" H 3650 4600 50  0001 C CNN
-F 3 "http://www.ti.com/lit/ds/symlink/tlv9064.pdf" H 3750 4700 50  0001 C CNN
-	2    3700 4500
-	1    0    0    -1
-$EndComp
-NoConn ~ 4000 4500
+P 3550 5300
+F 0 "U3" H 3550 5667 50  0000 C CNN
+F 1 "TLV9064IRTER" H 3550 5576 50  0000 C CNN
+F 2 "Package_DFN_QFN:QFN-16-1EP_3x3mm_P0.5mm_EP1.7x1.7mm" H 3500 5400 50  0001 C CNN
+F 3 "http://www.ti.com/lit/ds/symlink/tlv9064.pdf" H 3600 5500 50  0001 C CNN
+	2    3550 5300
+	1    0    0    -1
+$EndComp
 Text GLabel 3350 7025 0    50   Input ~ 0
 3V3
@@
 L power:GND #PWR0110
 U 1 1 5E19D1C9
-P 3300 4650
-F 0 "#PWR0110" H 3300 4400 50  0001 C CNN
-F 1 "GND" H 3305 4477 50  0000 C CNN
-F 2 "" H 3300 4650 50  0001 C CNN
-F 3 "" H 3300 4650 50  0001 C CNN
-	1    3300 4650
+P 3050 5200
+F 0 "#PWR0110" H 3050 4950 50  0001 C CNN
+F 1 "GND" H 3055 5027 50  0000 C CNN
+F 2 "" H 3050 5200 50  0001 C CNN
+F 3 "" H 3050 5200 50  0001 C CNN
+	1    3050 5200
 	-1   0    0    -1
 $EndComp
@@
 	0    -1   -1   0
 $EndComp
+Wire Wire Line
+	3150 5550 3850 5550
+Wire Wire Line
+	3850 5550 3850 5300
+Wire Wire Line
+	3050 5200 3250 5200
+Wire Wire Line
+	4650 4400 4850 4400
+Connection ~ 4850 4400
 $EndSCHEMATC

Commit message: Update V3
Parts:
- removed C17: 8pF, Capacitor_SMD:C_0603_1608Metric, symbol Device:C_Small
- removed Y1: 32.768, Crystal:Crystal_SMD_G8-2Pin_3.2x1.5mm, symbol Device:Crystal
- added C11: 8pF, Capacitor_SMD:C_0603_1608Metric, symbol Device:C_Small
- added C8: 4.7uF, Capacitor_SMD:C_0805_2012Metric, symbol Device:C_Small
- added R22: 50, Resistor_SMD:R_0603_1608Metric, symbol Device:R_Small
- added Y1: 32.768, Crystal:Crystal_SMD_G8-2Pin_3.2x1.5mm, symbol Device:Crystal_Small
- R10, R9: value 27 -> 50
- R21: value 85 -> 50
Connections:
- net 3V3: now also C8.2
- net BUTTONDOWN: now also U7.42 (PB6); no longer U7.41 (PB5)
- net BUTTONMID: now also U7.41 (PB5); no longer U7.40 (PB4)
- net BUTTONUP: now also U7.40 (PB4); no longer U7.39 (PB3)
- net GND: now also C16.2, C11.2, C8.1; no longer C16.1
- net LEDR: now also R22.1; no longer R21.1
- net VUSB: no longer U7.20 (PB2)
- net at U7.18 (PB0): now also TP2.1
- net at U7.3 (PC14): now also C11.1, Y1.2; no longer C16.2
- net at U7.38 (PA15): no longer TP2.1
- net at U7.4 (PC15): now also C16.1, Y1.1
- new net: R21.1, R22.2
- no-connect marks 20 -> 19
Other:
- moved on the sheet: C10, C6, C9, D1, D2, F1, R10, R21, R9, TP2, U5
